File: kicad/corfit.kicad_pcb (KiCad board)
At the start: 2 copper layers, 283.7 x 116.2 mm, 86 parts, among them J1 Conn_01x04_Pin, SW1 SW_PUSH, SW10 SW_PUSH, SW11 SW_PUSH, SW12 SW_PUSH, SW13 SW_PUSH, SW14 SW_PUSH, SW15 SW_PUSH, SW16 SW_PUSH, SW17 SW_PUSH, SW18 SW_PUSH, SW19 SW_PUSH, SW2 SW_PUSH, SW20 SW_PUSH, SW21 SW_PUSH, SW22 SW_PUSH, SW23 SW_PUSH, SW24 SW_PUSH, SW25 SW_PUSH, SW26 SW_PUSH, SW27 SW_PUSH, SW28 SW_PUSH, SW29 SW_PUSH, SW3 SW_PUSH, SW30 SW_PUSH, SW31 SW_PUSH, SW32 SW_PUSH, SW33 SW_PUSH, SW34 SW_PUSH, SW35 SW_PUSH, SW36 SW_PUSH, SW37 SW_PUSH, SW38 SW_PUSH, SW39 SW_PUSH, SW4 SW_PUSH, SW40 SW_PUSH, SW41 SW_PUSH, SW42 SW_PUSH, SW5 SW_PUSH, SW6 SW_PUSH, SW7 SW_PUSH, SW8 SW_PUSH, SW9 SW_PUSH, U1 RP2040-Zero

Commit message: feat: update the v1.0 PCB and add top and bottom plates
Parts:
- added Ref**: M2_SpacerHole, isw-kbd.pretty:M2_SpacerHole, F.Cu at (50.4, 68.7)
- added Ref**: M2_SpacerHole, isw-kbd.pretty:M2_SpacerHole, F.Cu at (284.2, 68.7)
- added Ref**: M2_SpacerHole, isw-kbd.pretty:M2_SpacerHole, F.Cu at (200.6, 119.5)
- added Ref**: M2_SpacerHole, isw-kbd.pretty:M2_SpacerHole, F.Cu at (242.6, 107.0)
- added Ref**: M2_SpacerHole, isw-kbd.pretty:M2_SpacerHole, F.Cu at (204.6, 67.5)
- added Ref**: M2_SpacerHole, isw-kbd.pretty:M2_SpacerHole, F.Cu at (130.0, 67.5)
- added Ref**: M2_SpacerHole, isw-kbd.pretty:M2_SpacerHole, F.Cu at (92.0, 107.0)
- added Ref**: M2_SpacerHole, isw-kbd.pretty:M2_SpacerHole, F.Cu at (134.0, 119.5)
- added Ref**: M2_SpacerHole, isw-kbd.pretty:M2_SpacerHole, F.Cu at (55.3, 50.2)
- added Ref**: M2_SpacerHole, isw-kbd.pretty:M2_SpacerHole, F.Cu at (279.3, 50.2)
- moved J1 1.08 mm to (167.3, 96.5)
Routing:
- net col7: track 120.1 -> 129.1 mm
- net col11: track 155.2 -> 159.9 mm
- net col1: track 154.3 -> 159.0 mm
- net col0: track 170.4 -> 168.3 mm
- net row1: track 285.0 -> 286.3 mm
- net col5: track 109.9 -> 111.1 mm
Other:
- board size 283.7 x 116.2 mm -> 283.9 x 116.2 mm
